Commit message: update to camera in my_robot.gazebo, my_robot.xacro. Added mapping.launch file.

File: catkin_ws/src/my_robot/urdf/my_robot.xacro (robot description, xacro)
@@ -125,4 +125,6 @@
     </visual>
   </link>
+  <link name="camera_link_optical">
+  </link>
     <link name ="hokuyo">
     <inertial>
@@ -176,3 +178,8 @@
     <axis xyz="0 1 0"/>
   </joint>
+  <joint name="camera_optical_joint" type="fixed">
+    <origin xyz="0 0 0" rpy="-1.5707 0 -1.5707"/>
+    <parent link="camera_link"/>
+    <child link="camera_link_optical"/>
+  </joint>
 </robot>

Commit message: fixed camera view

File: catkin_ws/src/my_robot/urdf/my_robot.xacro (robot description, xacro)
@@ -179,5 +179,5 @@
   </joint>
   <joint name="camera_optical_joint" type="fixed">
-    <origin xyz="0 0 0" rpy="-1.5707 0 -1.5707"/>
+    <origin xyz="0 0 0" rpy="0 0 0"/>
     <parent link="camera"/>
     <child link="camera_link_optical"/>
